File: pcb/connector.kicad_pcb (KiCad board)
At the start: 2 copper layers, 51.8 x 7.8 mm, 5 parts

Commit message: connector 0.3
Other:
- board text added: "v0.3"
- board text removed: "v0.2"
Changed lines of the file:
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@@
     (pad "" smd rect (at 0 -8.2 90) (size 2.5 2.5) (layers "F.Cu" "F.Paste" "F.Mask"))
     (pad "" smd rect (at 0 8.2 90) (size 2.5 2.5) (layers "F.Cu" "F.Paste" "F.Mask"))
-    (pad "1" smd rect (at -1.7 -5.5 90) (size 1.8 0.5) (layers "F.Cu" "F.Paste" "F.Mask")
+    (pad "1" smd rect (at -1.7 -5.5 90) (size 1.8 0.8) (layers "F.Cu" "F.Paste" "F.Mask")
       (net 1 "Net-(VIK_K1-3V3)") (pinfunction "3V3") (pintype "power_in") (thermal_bridge_angle 45))
-    (pad "2" smd rect (at 1.7 -4.5 90) (size 1.8 0.5) (layers "F.Cu" "F.Paste" "F.Mask")
+    (pad "2" smd rect (at 1.7 -4.5 90) (size 1.8 0.8) (layers "F.Cu" "F.Paste" "F.Mask")
       (net 2 "Net-(VIK_K1-GND-Pad2)") (pinfunction "GND") (pintype "power_in") (thermal_bridge_angle 45))
-    (pad "3" smd rect (at -1.7 -3.5 90) (size 1.8 0.5) (layers "F.Cu" "F.Paste" "F.Mask")
+    (pad "3" smd rect (at -1.7 -3.5 90) (size 1.8 0.8) (layers "F.Cu" "F.Paste" "F.Mask")
       (net 3 "Net-(VIK_K1-SDA)") (pinfunction "SDA") (pintype "bidirectional") (thermal_bridge_angle 45))
-    (pad "4" smd rect (at 1.7 -2.5 90) (size 1.8 0.5) (layers "F.Cu" "F.Paste" "F.Mask")
+    (pad "4" smd rect (at 1.7 -2.5 90) (size 1.8 0.8) (layers "F.Cu" "F.Paste" "F.Mask")
       (net 4 "Net-(VIK_K1-SCL)") (pinfunction "SCL") (pintype "bidirectional") (thermal_bridge_angle 45))
-    (pad "5" smd rect (at -1.7 -1.5 90) (size 1.7 0.5) (layers "F.Cu" "F.Paste" "F.Mask")
+    (pad "5" smd rect (at -1.7 -1.5 90) (size 1.7 0.8) (layers "F.Cu" "F.Paste" "F.Mask")
       (net 5 "Net-(VIK_K1-RGB_IN)") (pinfunction "RGB_IN") (pintype "input") (thermal_bridge_angle 45))
-    (pad "6" smd rect (at 1.7 -0.5 90) (size 1.8 0.5) (layers "F.Cu" "F.Paste" "F.Mask")
+    (pad "6" smd rect (at 1.7 -0.5 90) (size 1.8 0.8) (layers "F.Cu" "F.Paste" "F.Mask")
       (net 6 "Net-(VIK_K1-5V)") (pinfunction "5V") (pintype "power_in") (thermal_bridge_angle 45))
-    (pad "7" smd rect (at -1.7 0.5 90) (size 1.8 0.5) (layers "F.Cu" "F.Paste" "F.Mask")
+    (pad "7" smd rect (at -1.7 0.5 90) (size 1.8 0.8) (layers "F.Cu" "F.Paste" "F.Mask")
       (net 7 "Net-(VIK_K1-GND-Pad7)") (pinfunction "GND") (pintype "power_in"))
-    (pad "8" smd rect (at 1.7 1.5 90) (size 1.8 0.5) (layers "F.Cu" "F.Paste" "F.Mask")
+    (pad "8" smd rect (at 1.7 1.5 90) (size 1.8 0.8) (layers "F.Cu" "F.Paste" "F.Mask")
       (net 8 "Net-(VIK_K1-MOSI)") (pinfunction "MOSI") (pintype "input") (thermal_bridge_angle 45))
-    (pad "9" smd rect (at -1.7 2.5 90) (size 1.8 0.5) (layers "F.Cu" "F.Paste" "F.Mask")
+    (pad "9" smd rect (at -1.7 2.5 90) (size 1.8 0.8) (layers "F.Cu" "F.Paste" "F.Mask")
       (net 9 "Net-(VIK_K1-GPIO)") (pinfunction "GPIO") (pintype "bidirectional") (thermal_bridge_angle 45))
-    (pad "10" smd rect (at 1.7 3.5 90) (size 1.8 0.5) (layers "F.Cu" "F.Paste" "F.Mask")
+    (pad "10" smd rect (at 1.7 3.5 90) (size 1.8 0.8) (layers "F.Cu" "F.Paste" "F.Mask")
       (net 10 "Net-(VIK_K1-CS)") (pinfunction "CS") (pintype "input") (thermal_bridge_angle 45))
-    (pad "11" smd rect (at -1.7 4.5 90) (size 1.8 0.5) (layers "F.Cu" "F.Paste" "F.Mask")
+    (pad "11" smd rect (at -1.7 4.5 90) (size 1.8 0.8) (layers "F.Cu" "F.Paste" "F.Mask")
       (net 11 "Net-(VIK_K1-MISO)") (pinfunction "MISO") (pintype "output") (thermal_bridge_angle 45))
-    (pad "12" smd rect (at 1.7 5.5 90) (size 1.8 0.5) (layers "F.Cu" "F.Paste" "F.Mask")
+    (pad "12" smd rect (at 1.7 5.5 90) (size 1.8 0.8) (layers "F.Cu" "F.Paste" "F.Mask")
       (net 12 "Net-(VIK_K1-SCLK)") (pinfunction "SCLK") (pintype "input") (thermal_bridge_angle 45))
     (model "${ZZKEEB}/models/FPC vertical connector-1mm-10PIN.STEP" hide
-      (offset (xyz -1.2 8.5 0))
+      (offset (xyz 1.2 -8.5 0))
       (scale (xyz 1.1 1 1))
-      (rotate (xyz 0 0 90))
+      (rotate (xyz 0 0 -90))
     )
   )
@@
         (effects (font (size 1 1) (thickness 0.15)))
     )
-    (pad "" thru_hole circle (at 0 0) (size 4 4) (drill 2.3) (layers "*.Cu" "*.Mask"))
+    (pad "" thru_hole circle (at 0 0) (size 4.5 4.5) (drill 2.5) (layers "*.Cu" "*.Mask"))
   )
   (footprint "zzkeeb:Hole_M2-TH" (layer "B.Cu")
@@
         (effects (font (size 1 1) (thickness 0.15)) (justify mirror))
     )
-    (pad "" thru_hole circle (at 0 0 180) (size 4 4) (drill 2.3) (layers "*.Cu" "*.Mask"))
+    (pad "" thru_hole circle (at 0 0 180) (size 4.5 4.5) (drill 2.5) (layers "*.Cu" "*.Mask"))
   )
   (footprint "zzkeeb:Connector_FFC-12pin-1mm-vertical" (layer "B.Cu")
@@
     (pad "" smd rect (at 0 -8.2 270) (size 2.5 2.5) (layers "B.Cu" "B.Paste" "B.Mask"))
     (pad "" smd rect (at 0 8.2 270) (size 2.5 2.5) (layers "B.Cu" "B.Paste" "B.Mask"))
-    (pad "1" smd rect (at -1.7 5.5 270) (size 1.8 0.5) (layers "B.Cu" "B.Paste" "B.Mask")
+    (pad "1" smd rect (at -1.7 5.5 270) (size 1.8 0.8) (layers "B.Cu" "B.Paste" "B.Mask")
       (net 1 "Net-(VIK_K1-3V3)") (pinfunction "3V3") (pintype "power_in") (thermal_bridge_angle 45))
-    (pad "2" smd rect (at 1.7 4.5 270) (size 1.8 0.5) (layers "B.Cu" "B.Paste" "B.Mask")
+    (pad "2" smd rect (at 1.7 4.5 270) (size 1.8 0.8) (layers "B.Cu" "B.Paste" "B.Mask")
       (net 2 "Net-(VIK_K1-GND-Pad2)") (pinfunction "GND") (pintype "power_in") (thermal_bridge_angle 45))
-    (pad "3" smd rect (at -1.7 3.5 270) (size 1.8 0.5) (layers "B.Cu" "B.Paste" "B.Mask")
+    (pad "3" smd rect (at -1.7 3.5 270) (size 1.8 0.8) (layers "B.Cu" "B.Paste" "B.Mask")
       (net 3 "Net-(VIK_K1-SDA)") (pinfunction "SDA") (pintype "bidirectional") (thermal_bridge_angle 45))
-    (pad "4" smd rect (at 1.7 2.5 270) (size 1.8 0.5) (layers "B.Cu" "B.Paste" "B.Mask")
+    (pad "4" smd rect (at 1.7 2.5 270) (size 1.8 0.8) (layers "B.Cu" "B.Paste" "B.Mask")
       (net 4 "Net-(VIK_K1-SCL)") (pinfunction "SCL") (pintype "bidirectional") (thermal_bridge_angle 45))
-    (pad "5" smd rect (at -1.7 1.5 270) (size 1.7 0.5) (layers "B.Cu" "B.Paste" "B.Mask")
+    (pad "5" smd rect (at -1.7 1.5 270) (size 1.7 0.8) (layers "B.Cu" "B.Paste" "B.Mask")
       (net 5 "Net-(VIK_K1-RGB_IN)") (pinfunction "RGB_IN") (pintype "input") (thermal_bridge_angle 45))
-    (pad "6" smd rect (at 1.7 0.5 270) (size 1.8 0.5) (layers "B.Cu" "B.Paste" "B.Mask")
+    (pad "6" smd rect (at 1.7 0.5 270) (size 1.8 0.8) (layers "B.Cu" "B.Paste" "B.Mask")
       (net 6 "Net-(VIK_K1-5V)") (pinfunction "5V") (pintype "power_in") (thermal_bridge_angle 45))
-    (pad "7" smd rect (at -1.7 -0.5 270) (size 1.8 0.5) (layers "B.Cu" "B.Paste" "B.Mask")
+    (pad "7" smd rect (at -1.7 -0.5 270) (size 1.8 0.8) (layers "B.Cu" "B.Paste" "B.Mask")
       (net 7 "Net-(VIK_K1-GND-Pad7)") (pinfunction "GND") (pintype "power_in"))
-    (pad "8" smd rect (at 1.7 -1.5 270) (size 1.8 0.5) (layers "B.Cu" "B.Paste" "B.Mask")
+    (pad "8" smd rect (at 1.7 -1.5 270) (size 1.8 0.8) (layers "B.Cu" "B.Paste" "B.Mask")
       (net 8 "Net-(VIK_K1-MOSI)") (pinfunction "MOSI") (pintype "input") (thermal_bridge_angle 45))
-    (pad "9" smd rect (at -1.7 -2.5 270) (size 1.8 0.5) (layers "B.Cu" "B.Paste" "B.Mask")
+    (pad "9" smd rect (at -1.7 -2.5 270) (size 1.8 0.8) (layers "B.Cu" "B.Paste" "B.Mask")
       (net 9 "Net-(VIK_K1-GPIO)") (pinfunction "GPIO") (pintype "bidirectional") (thermal_bridge_angle 45))
-    (pad "10" smd rect (at 1.7 -3.5 270) (size 1.8 0.5) (layers "B.Cu" "B.Paste" "B.Mask")
+    (pad "10" smd rect (at 1.7 -3.5 270) (size 1.8 0.8) (layers "B.Cu" "B.Paste" "B.Mask")
       (net 10 "Net-(VIK_K1-CS)") (pinfunction "CS") (pintype "input") (thermal_bridge_angle 45))
-    (pad "11" smd rect (at -1.7 -4.5 270) (size 1.8 0.5) (layers "B.Cu" "B.Paste" "B.Mask")
+    (pad "11" smd rect (at -1.7 -4.5 270) (size 1.8 0.8) (layers "B.Cu" "B.Paste" "B.Mask")
       (net 11 "Net-(VIK_K1-MISO)") (pinfunction "MISO") (pintype "output") (thermal_bridge_angle 45))
-    (pad "12" smd rect (at 1.7 -5.5 270) (size 1.8 0.5) (layers "B.Cu" "B.Paste" "B.Mask")
+    (pad "12" smd rect (at 1.7 -5.5 270) (size 1.8 0.8) (layers "B.Cu" "B.Paste" "B.Mask")
       (net 12 "Net-(VIK_K1-SCLK)") (pinfunction "SCLK") (pintype "input") (thermal_bridge_angle 45))
     (model "${ZZKEEB}/models/FPC vertical connector-1mm-10PIN.STEP"
@@
     )
   )
-  (gr_circle (center 101.783 85.316) (end 102.283 85.316)
-    (stroke (width 0.1) (type solid)) (fill solid) (layer "B.SilkS"))
-  (gr_circle (center 101.783 79.716) (end 102.283 79.716)
-    (stroke (width 0.1) (type solid)) (fill solid) (layer "F.SilkS"))
   (gr_line (start 152.483 85.416) (end 152.483 79.616)
     (stroke (width 0.1) (type default)) (layer "Edge.Cuts"))
@@
   (gr_line (start 151.483 78.616) (end 101.683 78.616)
     (stroke (width 0.1) (type default)) (layer "Edge.Cuts"))
-  (gr_text "v0.2" (at 149.583 79.516) (layer "B.SilkS")
+  (gr_text "v0.3" (at 103.583 85.516 180) (layer "B.SilkS")
     (effects (font (size 1 1) (thickness 0.15)) (justify mirror))
   )
-  (gr_text "v0.2" (at 149.583 79.516) (layer "F.SilkS")
+  (gr_text "v0.3" (at 103.583 85.516 180) (layer "F.SilkS")
     (effects (font (size 1 1) (thickness 0.15)))
   )
