File: pcb/connector.kicad_pcb (KiCad board)
At the start: 2 copper layers, 51.8 x 7.8 mm, 5 parts

Commit message: final PCBs
Other:
- board text added: "JLCJLCJLCJLC"
- board text added: "v1.0"
- board text removed: "v0.3"
Changed lines of the file:
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@@
   (gr_line (start 151.483 78.616) (end 101.683 78.616)
     (stroke (width 0.1) (type default)) (layer "Edge.Cuts"))
-  (gr_text "v0.3" (at 103.583 85.516 180) (layer "B.SilkS")
+  (gr_text "v1.0" (at 103.583 85.516 180) (layer "B.SilkS")
     (effects (font (size 1 1) (thickness 0.15)) (justify mirror))
   )
-  (gr_text "v0.3" (at 103.583 85.516 180) (layer "F.SilkS")
+  (gr_text "JLCJLCJLCJLC" (at 143.083 79.516 180) (layer "F.SilkS")
+    (effects (font (size 0.8 0.8) (thickness 0.15)))
+  )
+  (gr_text "v1.0" (at 103.583 85.516 180) (layer "F.SilkS")
     (effects (font (size 1 1) (thickness 0.15)))
   )
