File: pcb/pcb.kicad_pcb (KiCad board)
At the start: 2 copper layers, 165.5 x 101.1 mm, 59 parts, among them J1 N!N, J2 Conn_01x02_Socket, J4 Display_nice-view, J8 Conn_01x12_Socket, J9 Conn_01x12_Socket, SW1 Switch, SW10 Switch, SW11 Switch, SW12 Switch, SW13 Switch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

Commit message: small updates
Parts:
- moved SW21 3.50 mm to (164.8, 53.9)

Commit message: move mcu to right, add encoder
Parts:
- removed S2: Button_5way-SKRHABE010, zzkeeb:Button_5way-SKRHABE010
- added SW23: RotaryEncoder_Switch, zzkeeb:RotaryEncoder_EC11, B.Cu at (98.5, 110.0)
- D1, D10, D11, D12, D13, D14, D15, D16, D17, D18, D19, D2, D20, D3, D4, D5, D6, D7, D8, D9: footprint zzkeeb:Diode_1N4148-SOD123-reversible-flip3d -> zzkeeb:Diode_1N4148-SOD123-reversible
- J1, J2, SW21, SW22: moved to F.Cu
- SW1, SW10, SW11, SW12, SW13, SW14, SW15, SW16, SW17, SW18, SW19, SW2, SW20, SW3, SW4, SW5, SW6, SW7, SW8, SW9: footprint zzkeeb:Switch_ChocV1-hotswap-reversible -> zzkeeb:Switch_ChocV1-hotswap-reversible-flip3d
- moved J2 3.50 mm to (173.6, 103.1), turned to -160 degrees
- turned SW22 to -160 degrees
- turned J1 to 20 degrees
- turned S1 to -90 degrees
Connections:
- J1 pad 10: col2_r -> col6
- J1 pad 11: col1_r -> col5
- J1 pad 12: col0_r -> row1
- J1 pad 13: row2 -> col0
- J1 pad 14: row1 -> col1
- J1 pad 15: row0 -> col2
- J1 pad 16: col4 -> col3
- J1 pad 17: col3 -> col4
- J1 pad 18: col2 -> row4
- J1 pad 19: col1 -> row3
- J1 pad 2: row4 -> row0
- J1 pad 20: col0 -> row2
- J1 pad 7: row3 -> col9
- J1 pad 8: col4_r -> col8
- J1 pad 9: col3_r -> col7
- J8 pad 10: col2 -> col7
- J8 pad 11: col3 -> col6
- J8 pad 12: col4 -> col5
- J8 pad 8: col0 -> col9
- J8 pad 9: col1 -> col8
- J9 pad 10: col2_r -> col2
- J9 pad 11: col3_r -> col3
- J9 pad 12: col4_r -> col4
- J9 pad 8: col0_r -> col0
- J9 pad 9: col1_r -> col1
- S1 pad 1: col0 -> col9
- S1 pad 2: col4 -> col5
- S1 pad 3: col2 -> col7
- S1 pad 4: col1 -> col8
- S1 pad 6: col3 -> col6
- SW1 pad 2: col0 -> col9
- SW10 pad 2: col4 -> col5
- SW11 pad 2: col0 -> col9
- SW12 pad 2: col1 -> col8
- SW13 pad 2: col2 -> col7
- SW14 pad 2: col3 -> col6
- SW15 pad 2: col4 -> col5
- SW16 pad 2: col0 -> col9
- SW17 pad 2: col1 -> col8
- SW18 pad 2: col2 -> col7
- SW19 pad 2: col3 -> col6
- SW2 pad 2: col1 -> col8
- SW20 pad 2: col4 -> col5
- SW3 pad 2: col2 -> col7
- SW4 pad 2: col3 -> col6
- SW5 pad 2: col4 -> col5
- SW6 pad 2: col0 -> col9
- SW7 pad 2: col1 -> col8
- SW8 pad 2: col2 -> col7
- SW9 pad 2: col3 -> col6
Routing:
- net col8: track 0.00 -> 310.5 mm, vias 0 -> 7
- net col9: track 0.00 -> 305.7 mm, vias 0 -> 7
- net col1: track 313.0 -> 40.0 mm, vias 7 -> 0
- net col0: track 307.4 -> 38.2 mm, vias 7 -> 0
- net col6: track 0.00 -> 269.0 mm, vias 0 -> 8
- net col5: track 0.00 -> 255.1 mm, vias 0 -> 6
- net col7: track 0.00 -> 251.8 mm, vias 0 -> 7
- net col3: track 270.4 -> 43.6 mm, vias 8 -> 0
- net col2: track 256.1 -> 41.8 mm, vias 7 -> 0
- net col4: track 256.1 -> 45.4 mm, vias 7 -> 0
- net encA: track 0.00 -> 115.4 mm, vias 0 -> 2
- net encB: track 0.00 -> 111.6 mm, vias 0 -> 2
- net GND: track 178.6 -> 257.4 mm, vias 1 -> 3
- net col4_r: track 47.3 -> 0.00 mm
- net col3_r: track 45.5 -> 0.00 mm
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Other:
- outline, holes or cut-outs redrawn
- board text added: "C5"
- board text added: "C6"
- board text added: "R4"
- board text added: "encA"
- board text added: "encB"
- board text removed: "nice!nano"
- board text removed: "nice!view"

Commit message: 0.2
Other:
- board text added: "JLCJLCJLCJLC"
Changed lines of the file:
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@@
     (effects (font (size 0.8 0.8) (thickness 0.15)) (justify left))
+  )
+  (gr_text "JLCJLCJLCJLC" (at 48.5 66) (layer "F.SilkS")
+    (effects (font (size 0.8 0.8) (thickness 0.15)))
   )
   (gr_text "encB" (at 86.8 107.5) (layer "F.SilkS")

Commit message: pcb 0.3
Parts:
- D1, D10, D11, D12, D13, D14, D15, D16, D17, D18, D19, D2, D20, D3, D4, D5, D6, D7, D8, D9: footprint zzkeeb:Diode_1N4148-SOD123-reversible -> zzkeeb:Diode_1N4148-SOD123-reversible-flip3d
- J4, J9: moved to B.Cu
- J8: moved to F.Cu
- SW1, SW10, SW11, SW12, SW13, SW14, SW15, SW16, SW17, SW18, SW19, SW2, SW20, SW3, SW4, SW5, SW6, SW7, SW8, SW9: footprint zzkeeb:Switch_ChocV1-hotswap-reversible-flip3d -> zzkeeb:Switch_ChocV1-hotswap-reversible
- turned J4 to -160 degrees
- turned J8 to 110 degrees
- turned J9 to -70 degrees
Connections:
- J1 pad 18: row4 -> row2
- J1 pad 20: row2 -> row4
- J8 pad 3: row0 -> row4
- J8 pad 4: row1 -> row3
- J8 pad 6: row3 -> row1
- J8 pad 7: row4 -> row0
- J9 pad 1: BAT -> col4
- J9 pad 10: col2 -> row4
- J9 pad 11: col3 -> GND
- J9 pad 12: col4 -> BAT
- J9 pad 2: GND -> col3
- J9 pad 3: row0 -> col2
- J9 pad 4: row1 -> col1
- J9 pad 5: row2 -> col0
- J9 pad 6: row3 -> row0
- J9 pad 7: row4 -> row1
- J9 pad 8: col0 -> row2
- J9 pad 9: col1 -> row3
Routing:
- net row0: track 216.1 -> 180.7 mm
- net GND: track 257.4 -> 238.1 mm, vias 3 -> 2
- net BAT: track 100.9 -> 86.1 mm
- net col5: track 255.1 -> 240.3 mm, vias 6 -> 5
- net col6: track 269.0 -> 256.5 mm, vias 8 -> 7
- net col7: track 251.8 -> 241.7 mm, vias 7 -> 6
- net col8: track 310.5 -> 302.5 mm, vias 7 -> 6
- net row1: track 162.8 -> 155.6 mm
- net encB: track 111.6 -> 118.9 mm
- net encA: track 115.4 -> 122.4 mm
- net row3: track 246.3 -> 253.0 mm
- net +3.3V: track 43.3 -> 49.9 mm
- net CS: track 67.6 -> 73.9 mm
- net col9: track 305.7 -> 300.2 mm, vias 7 -> 6
- net row4: track 175.7 -> 180.0 mm, vias 1 -> 2
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Other:
- board text added: "v0.3"
- board text removed: "v0.2"

Commit message: final PCBs
Other:
- board text added: "v1.0"
- board text removed: "BATTERY"
- board text removed: "v0.3"
